File: pcb/SMD-Challenge-Avanti.kicad_pcb (KiCad board)
At the start: 2 copper layers, 72.9 x 101.2 mm, 16 parts, among them SW1 SW_SPDT, U1 SN74LVC1G14DBV, U2 74HC4017

Commit message: Fix blink order
Connections:
- U2 pad 2: Net-(D3-A) -> Net-(D4-A)
- U2 pad 3: Net-(D4-A) -> Net-(D3-A)
Routing:
- net Net-(D4-A): track 78.3 -> 79.9 mm
Other:
- board text added: "v2.0.1"
- board text removed: "v2.0.0"
Changed lines of the file:
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@@
     (title "SMD-Challenge-Avanti")
     (date "2023-01-30")
-    (rev "v2.0.0")
+    (rev "v2.0.1")
     (company "(c) by C. Zaugg")
     (comment 1 "Made for Avanti 2023")
@@
       (net 7 "Net-(D2-A)") (pinfunction "Q5") (pintype "output"))
     (pad "2" smd roundrect (at -2.575 3.175 180) (size 1.75 0.6) (layers "B.Cu" "B.Paste" "B.Mask") (roundrect_rratio 0.25)
-      (net 8 "Net-(D3-A)") (pinfunction "Q1") (pintype "output"))
+      (net 9 "Net-(D4-A)") (pinfunction "Q1") (pintype "output"))
     (pad "3" smd roundrect (at -2.575 1.905 180) (size 1.75 0.6) (layers "B.Cu" "B.Paste" "B.Mask") (roundrect_rratio 0.25)
-      (net 9 "Net-(D4-A)") (pinfunction "Q0") (pintype "output"))
+      (net 8 "Net-(D3-A)") (pinfunction "Q0") (pintype "output"))
     (pad "4" smd roundrect (at -2.575 0.635 180) (size 1.75 0.6) (layers "B.Cu" "B.Paste" "B.Mask") (roundrect_rratio 0.25)
       (net 10 "Net-(D5-A)") (pinfunction "Q2") (pintype "output"))
@@
       (net 12 "Net-(U2-Q6)") (pinfunction "Q6") (pintype "output"))
     (pad "6" smd roundrect (at -2.575 -1.905 180) (size 1.75 0.6) (layers "B.Cu" "B.Paste" "B.Mask") (roundrect_rratio 0.25)
-      (net 13 "unconnected-(U2-Q7-Pad6)") (pinfunction "Q7") (pintype "output"))
+      (net 13 "unconnected-(U2-Q7-Pad6)") (pinfunction "Q7") (pintype "output+no_connect"))
     (pad "7" smd roundrect (at -2.575 -3.175 180) (size 1.75 0.6) (layers "B.Cu" "B.Paste" "B.Mask") (roundrect_rratio 0.25)
       (net 11 "Net-(D6-A)") (pinfunction "Q3") (pintype "output"))
@@
       (net 2 "GND") (pinfunction "VSS") (pintype "power_in"))
     (pad "9" smd roundrect (at 2.575 -4.445 180) (size 1.75 0.6) (layers "B.Cu" "B.Paste" "B.Mask") (roundrect_rratio 0.25)
-      (net 14 "unconnected-(U2-Q8-Pad9)") (pinfunction "Q8") (pintype "output"))
+      (net 14 "unconnected-(U2-Q8-Pad9)") (pinfunction "Q8") (pintype "output+no_connect"))
     (pad "10" smd roundrect (at 2.575 -3.175 180) (size 1.75 0.6) (layers "B.Cu" "B.Paste" "B.Mask") (roundrect_rratio 0.25)
       (net 6 "Net-(D1-A)") (pinfunction "Q4") (pintype "output"))
     (pad "11" smd roundrect (at 2.575 -1.905 180) (size 1.75 0.6) (layers "B.Cu" "B.Paste" "B.Mask") (roundrect_rratio 0.25)
-      (net 15 "unconnected-(U2-Q9-Pad11)") (pinfunction "Q9") (pintype "output"))
+      (net 15 "unconnected-(U2-Q9-Pad11)") (pinfunction "Q9") (pintype "output+no_connect"))
     (pad "12" smd roundrect (at 2.575 -0.635 180) (size 1.75 0.6) (layers "B.Cu" "B.Paste" "B.Mask") (roundrect_rratio 0.25)
       (net 18 "unconnected-(U2-Cout-Pad12)") (pinfunction "Cout") (pintype "output+no_connect"))
@@
   (gr_line (start 170.522266 141.365008) (end 170.62361 141.066725)
     (stroke (width 0.264583) (type solid)) (layer "Edge.Cuts"))
-  (gr_text "v2.0.0" (at 125.9 131.9 110) (layer "B.Cu")
+  (gr_text "v2.0.1" (at 125.9 131.9 110) (layer "B.Cu")
     (effects (font (size 0.8 0.8) (thickness 0.15)) (justify mirror))
   )
@@
   (arc (start 150.44478 68.555) (mid 154.694827 67.709613) (end 158.297843 65.302156) (width 0.4) (layer "B.Cu") (net 7))
   (segment (start 174.988101 108.33125) (end 170.413456 104.500984) (width 0.4) (layer "F.Cu") (net 8))
-  (segment (start 166.533187 95.133187) (end 156.404162 85.004163) (width 0.4) (layer "F.Cu") (net 8))
-  (via (at 156.5 85.1) (size 0.8) (drill 0.4) (layers "F.Cu" "B.Cu") (net 8))
+  (segment (start 157.664213 86.264214) (end 166.533187 95.133187) (width 0.4) (layer "F.Cu") (net 8))
+  (via (at 154.25 84.85) (size 0.8) (drill 0.4) (layers "F.Cu" "B.Cu") (net 8))
   (arc (start 168.8 100.605757) (mid 168.210874 97.644023) (end 166.533187 95.133187) (width 0.4) (layer "F.Cu") (net 8))
+  (arc (start 154.25 84.85) (mid 156.097759 85.217542) (end 157.664213 86.264214) (width 0.4) (layer "F.Cu") (net 8))
   (arc (start 170.413456 104.500984) (mid 169.219323 102.713839) (end 168.8 100.605757) (width 0.4) (layer "F.Cu") (net 8))
-  (segment (start 148.375 69.825) (end 150.213956 69.825) (width 0.4) (layer "B.Cu") (net 8))
-  (segment (start 153.6 73.211044) (end 153.6 78.098781) (width 0.4) (layer "B.Cu") (net 8))
-  (arc (start 153.6 78.098781) (mid 154.353686 81.887814) (end 156.5 85.1) (width 0.4) (layer "B.Cu") (net 8))
-  (arc (start 150.213956 69.825) (mid 152.608251 70.816749) (end 153.6 73.211044) (width 0.4) (layer "B.Cu") (net 8))
+  (segment (start 149.905913 71.095) (end 148.375 71.095) (width 0.4) (layer "B.Cu") (net 8))
+  (segment (start 152.4 83) (end 152.4 73.589087) (width 0.4) (layer "B.Cu") (net 8))
+  (arc (start 152.4 73.589087) (mid 151.669499 71.825501) (end 149.905913 71.095) (width 0.4) (layer "B.Cu") (net 8))
+  (arc (start 154.25 84.85) (mid 152.941852 84.308148) (end 152.4 83) (width 0.4) (layer "B.Cu") (net 8))
+  (segment (start 160.744458 140.556893) (end 161.021269 140.556893) (width 0.4) (layer "F.Cu") (net 9))
   (segment (start 158.5 137.179898) (end 158.5 137.827208) (width 0.4) (layer "F.Cu") (net 9))
   (segment (start 164.3 108.168917) (end 164.3 123.177461) (width 0.4) (layer "F.Cu") (net 9))
-  (segment (start 160.744458 140.556893) (end 161.021269 140.556893) (width 0.4) (layer "F.Cu") (net 9))
-  (segment (start 154.4 85.8) (end 155.483144 86.883144) (width 0.4) (layer "F.Cu") (net 9))
-  (via (at 154.4 85.8) (size 0.8) (drill 0.4) (layers "F.Cu" "B.Cu") (net 9))
-  (arc (start 159.9 133.8) (mid 158.863848 135.350711) (end 158.5 137.179898) (width 0.4) (layer "F.Cu") (net 9))
-  (arc (start 164.3 123.177461) (mid 163.156477 128.926338) (end 159.9 133.8) (width 0.4) (layer "F.Cu") (net 9))
-  (arc (start 155.483144 86.883144) (mid 162.008573 96.649139) (end 164.3 108.168917) (width 0.4) (layer "F.Cu") (net 9))
+  (via (at 155.483144 86.883144) (size 0.8) (drill 0.4) (layers "F.Cu" "B.Cu") (net 9))
   (arc (start 158.5 137.827208) (mid 158.733903 139.003115) (end 159.4 140) (width 0.4) (layer "F.Cu") (net 9))
+  (arc (start 155.483144 86.883144) (mid 162.008573 96.649139) (end 164.3 108.168917) (width 0.4) (layer "F.Cu") (net 9))
+  (arc (start 159.9 133.8) (mid 158.863848 135.350711) (end 158.5 137.179898) (width 0.4) (layer "F.Cu") (net 9))
   (arc (start 159.4 140) (mid 160.016843 140.412161) (end 160.744458 140.556893) (width 0.4) (layer "F.Cu") (net 9))
-  (segment (start 152.4 73.589087) (end 152.4 80.971573) (width 0.4) (layer "B.Cu") (net 9))
-  (segment (start 148.375 71.095) (end 149.905913 71.095) (width 0.4) (layer "B.Cu") (net 9))
-  (arc (start 149.905913 71.095) (mid 151.669499 71.825501) (end 152.4 73.589087) (width 0.4) (layer "B.Cu") (net 9))
-  (arc (start 152.4 80.971573) (mid 152.919783 83.584699) (end 154.4 85.8) (width 0.4) (layer "B.Cu") (net 9))
+  (arc (start 164.3 123.177461) (mid 163.156477 128.926338) (end 159.9 133.8) (width 0.4) (layer "F.Cu") (net 9))
+  (segment (start 155.483144 86.883144) (end 155.483144 84.732098) (width 0.4) (layer "B.Cu") (net 9))
+  (segment (start 150.213956 69.825) (end 148.375 69.825) (width 0.4) (layer "B.Cu") (net 9))
+  (segment (start 153.6 80.185787) (end 153.6 73.211044) (width 0.4) (layer "B.Cu") (net 9))
+  (arc (start 153.6 73.211044) (mid 152.608251 70.816749) (end 150.213956 69.825) (width 0.4) (layer "B.Cu") (net 9))
+  (arc (start 154.6 82.6) (mid 153.859892 81.49235) (end 153.6 80.185787) (width 0.4) (layer "B.Cu") (net 9))
+  (arc (start 155.483144 84.732098) (mid 155.253622 83.578215) (end 154.6 82.6) (width 0.4) (layer "B.Cu") (net 9))
   (segment (start 129 139.4) (end 128.795735 139.604266) (width 0.4) (layer "F.Cu") (net 10))
   (segment (start 136.6 87.6) (end 136.506602 87.693398) (width 0.4) (layer "F.Cu") (net 10))

Commit message: Fix text
Other:
- board text added: "AVANTI"
- board text removed: "AVANT"
Changed lines of the file:
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@@
     (effects (font (size 0.8 0.8) (thickness 0.15)) (justify mirror))
   )
-  (gr_text "AVANT" (at 124.2 124.4 97) (layer "B.Cu")
+  (gr_text "AVANTI" (at 124.2 124.3 97) (layer "B.Cu")
     (effects (font (size 0.8 0.8) (thickness 0.15)) (justify mirror))
   )
@@
     (effects (font (size 0.8 0.8) (thickness 0.15)) (justify mirror))
   )
-  (gr_text "FOR" (at 123.9 120.9 92) (layer "B.Cu")
+  (gr_text "FOR" (at 123.9 120.65 92) (layer "B.Cu")
     (effects (font (size 0.8 0.8) (thickness 0.15)) (justify mirror))
   )
