File: pcb/SMD-Challenge.kicad_pcb (KiCad board)
At the start: 2 copper layers, 0 parts

Commit message: Add first draft
Parts:
- added BT1: Battery_Cell, Battery:BatteryHolder_Keystone_3002_1x2032, B.Cu at (145.6, 99.6)
- added C1: 1u, Capacitor_SMD:C_1206_3216Metric, B.Cu at (148.2, 58.0)
- added D1: LED, LED_SMD:LED_1206_3216Metric, F.Cu at (162.4, 140.8)
- added D10: LED, LED_SMD:LED_0201_0603Metric, F.Cu at (140.2, 63.8)
- added D2: LED, LED_SMD:LED_1206_3216Metric, F.Cu at (125.6, 140.6)
- added D3: LED, LED_SMD:LED_0805_2012Metric, F.Cu at (114.4, 107.8)
- added D4: LED, LED_SMD:LED_0805_2012Metric, F.Cu at (175.8, 108.8)
- added D5: LED, LED_SMD:LED_0603_1608Metric, F.Cu at (162.6, 51.4)
- added D6: LED, LED_SMD:LED_0603_1608Metric, F.Cu at (128.8, 51.2)
- added D7: LED, LED_SMD:LED_0402_1005Metric, F.Cu at (151.6, 85.8)
- added D8: LED, LED_SMD:LED_0402_1005Metric, F.Cu at (140.5, 85.9)
- added D9: LED, LED_SMD:LED_0201_0603Metric, F.Cu at (151.0, 63.8)
- added R1: R, Resistor_SMD:R_1206_3216Metric, F.Cu at (155.0, 137.4)
- added R10: R, Resistor_SMD:R_0201_0603Metric, F.Cu at (140.2, 61.6)
- added R11: 10k, Resistor_SMD:R_1206_3216Metric, B.Cu at (148.2, 63.6)
- added R2: R, Resistor_SMD:R_1206_3216Metric, F.Cu at (134.2, 137.4)
- added R3: R, Resistor_SMD:R_0805_2012Metric, F.Cu at (119.0, 104.0)
- added R4: R, Resistor_SMD:R_0805_2012Metric, F.Cu at (171.0, 105.2)
- added R5: R, Resistor_SMD:R_0603_1608Metric, F.Cu at (165.6, 54.4)
- added R6: R, Resistor_SMD:R_0603_1608Metric, F.Cu at (126.0, 54.0)
- added R7: R, Resistor_SMD:R_0402_1005Metric, F.Cu at (149.2, 86.4)
- added R8: R, Resistor_SMD:R_0402_1005Metric, F.Cu at (143.0, 86.4)
- added R9: R, Resistor_SMD:R_0201_0603Metric, F.Cu at (151.0, 61.4)
- added REF**: MountingHole_2.2mm_M2, MountingHole:MountingHole_2.2mm_M2, F.Cu at (145.6, 51.4)
- added RV1: 100k, Potentiometer_SMD:Potentiometer_Bourns_TC33X_Vertical, B.Cu at (144.0, 63.6)
- added U1: SN74LVC1G14DBV, Package_TO_SOT_SMD:SOT-23-5, B.Cu at (144.0, 58.0)
- added U2: 4017, Package_SO:SO-16_3.9x9.9mm_P1.27mm, B.Cu at (145.8, 73.0)
- added kibuzzard-63D590DE: G***, kibuzzard-63D590DE, B.Cu at (146.0, 117.0)
- added kibuzzard-63D590F7: G***, kibuzzard-63D590F7, B.Cu at (145.0, 122.0)
Routing:
- net VCC: track 0.00 -> 205.5 mm, vias 0 -> 4
- net Net-(R1-Pad1): track 0.00 -> 75.5 mm, vias 0 -> 1
- net Net-(R2-Pad1): track 0.00 -> 68.0 mm, vias 0 -> 1
- net Net-(R3-Pad1): track 0.00 -> 50.4 mm, vias 0 -> 1
- net Net-(R4-Pad1): track 0.00 -> 41.4 mm, vias 0 -> 1
- net Net-(R6-Pad1): track 0.00 -> 29.9 mm, vias 0 -> 1
- net Net-(R5-Pad1): track 0.00 -> 24.7 mm, vias 0 -> 1
- net Net-(RV1-Pad1): track 0.00 -> 20.4 mm
- net Net-(R10-Pad1): track 0.00 -> 18.2 mm, vias 0 -> 1
- net Net-(R8-Pad1): track 0.00 -> 17.7 mm, vias 0 -> 1
- net Net-(R7-Pad1): track 0.00 -> 14.3 mm, vias 0 -> 1
- net Net-(R9-Pad1): track 0.00 -> 13.8 mm, vias 0 -> 1
- net Net-(C1-Pad1): track 0.00 -> 6.87 mm
- net Net-(D2-Pad2): track 0.00 -> 6.74 mm
- net Net-(D1-Pad2): track 0.00 -> 5.59 mm
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- added copper zone on B.Cu, net GND
- added copper zone on F.Cu, net GND
Other:
- board outline added: 72.9 x 101.2 mm
- board text added: "2023"
- board text added: "AVANT"
- board text added: "FOR"
- board text added: "v1.0.0"

Commit message: Updated design
Parts:
- removed R1, R2: R, Resistor_SMD:R_1206_3216Metric
- removed R10, R9: R, Resistor_SMD:R_0201_0603Metric
- removed R3, R4: R, Resistor_SMD:R_0805_2012Metric
- removed R5, R6: R, Resistor_SMD:R_0603_1608Metric
- removed R7, R8: R, Resistor_SMD:R_0402_1005Metric
- removed REF**: MountingHole_2.2mm_M2, MountingHole:MountingHole_2.2mm_M2
- added H1: MountingHole, MountingHole:MountingHole_2.2mm_M2, F.Cu at (145.6, 51.3)
- added SW1: SW_SPDT, Button_Switch_SMD:SW_SPDT_PCM12, B.Cu at (164.5, 90.3)
- moved D5 2.56 mm to (164.8, 52.6)
- moved D6 2.12 mm to (127.3, 52.7)
- moved D10 1.60 mm to (140.3, 62.2)
- moved D9 1.60 mm to (151.0, 62.2)
- moved D7 1.02 mm to (150.6, 86.0)
- moved D8 0.71 mm to (141.2, 86.1)
Connections:
- BT1 pad 1: VCC -> Net-(BT1-+)
- D1 pad 2: Net-(D1-Pad2) -> Net-(D1-A)
- D10 pad 2: Net-(D10-Pad2) -> Net-(D10-A)
- D2 pad 2: Net-(D2-Pad2) -> Net-(D2-A)
- D3 pad 2: Net-(D3-Pad2) -> Net-(D3-A)
- D4 pad 2: Net-(D4-Pad2) -> Net-(D4-A)
- D5 pad 2: Net-(D5-Pad2) -> Net-(D5-A)
- D6 pad 2: Net-(D6-Pad2) -> Net-(D6-A)
- D7 pad 2: Net-(D7-Pad2) -> Net-(D7-A)
- D8 pad 2: Net-(D8-Pad2) -> Net-(D8-A)
- D9 pad 2: Net-(D9-Pad2) -> Net-(D9-A)
- U2 pad 1: Net-(R5-Pad1) -> Net-(D5-A)
- U2 pad 10: Net-(R6-Pad1) -> Net-(D6-A)
- U2 pad 11: Net-(R1-Pad1) -> Net-(D1-A)
- U2 pad 2: Net-(R9-Pad1) -> Net-(D9-A)
- U2 pad 3: Net-(R10-Pad1) -> Net-(D10-A)
- U2 pad 4: Net-(R8-Pad1) -> Net-(D8-A)
- U2 pad 5: Net-(R4-Pad1) -> Net-(D4-A)
- U2 pad 6: Net-(R3-Pad1) -> Net-(D3-A)
- U2 pad 7: Net-(R7-Pad1) -> Net-(D7-A)
- U2 pad 9: Net-(R2-Pad1) -> Net-(D2-A)
Routing:
- net Net-(D1-A): track 0.00 -> 80.9 mm, vias 0 -> 1
- net Net-(R1-Pad1): track 75.5 -> 0.00 mm, vias 1 -> 0
- net Net-(D2-A): track 0.00 -> 72.1 mm, vias 0 -> 1
- net Net-(R2-Pad1): track 68.0 -> 0.00 mm, vias 1 -> 0
- net VCC: track 205.5 -> 137.8 mm
- net Net-(D3-A): track 0.00 -> 56.7 mm, vias 0 -> 1
- net Net-(R3-Pad1): track 50.4 -> 0.00 mm, vias 1 -> 0
- net Net-(BT1-+): track 0.00 -> 49.6 mm
- net Net-(D4-A): track 0.00 -> 46.2 mm, vias 0 -> 1
- net Net-(R4-Pad1): track 41.4 -> 0.00 mm, vias 1 -> 0
- net Net-(D6-A): track 0.00 -> 31.7 mm, vias 0 -> 1
- net Net-(R6-Pad1): track 29.9 -> 0.00 mm, vias 1 -> 0
- net Net-(D5-A): track 0.00 -> 26.2 mm, vias 0 -> 1
- net Net-(R5-Pad1): track 24.7 -> 0.00 mm, vias 1 -> 0
- net Net-(D8-A): track 0.00 -> 19.4 mm, vias 0 -> 1
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
Commit message: Fixed version 1
Other:
- board text added: "BAER"
- board text added: "MOSER"
- board text added: "v1.1.0"
- board text removed: "AVANT"
- board text removed: "FOR"
- board text removed: "v1.0.0"
Changed lines of the file:
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@@
     (title "SMD-Challenge")
     (date "2023-01-30")
-    (rev "v1.0.0")
+    (rev "v1.1.0")
     (company "(c) by C. Zaugg")
-    (comment 3 "Moser Baer branding")
+    (comment 3 "Moser Baer Branding")
     (comment 4 "SMD - Challenge Badge")
   )
@@
       (drillshape 0)
       (scaleselection 1)
-      (outputdirectory "../prod/")
+      (outputdirectory "../prod/SMD-Challenge-Gerber/")
     )
   )
@@
     (fp_line (start 1.6 0.8) (end 1.6 -0.8)
       (stroke (width 0.1) (type solid)) (layer "B.Fab"))
-    (pad "1" smd roundrect (at -1.475 0 90) (size 1.15 1.8) (layers "B.Cu" "B.Paste" "B.Mask") (roundrect_rratio 0.217391)
+    (pad "1" smd roundrect (at -1.475 0 90) (size 1.15 1.8) (layers "B.Cu" "B.Paste" "B.Mask") (roundrect_rratio 0.2173913043)
       (net 1 "Net-(C1-Pad1)") (pintype "passive"))
-    (pad "2" smd roundrect (at 1.475 0 90) (size 1.15 1.8) (layers "B.Cu" "B.Paste" "B.Mask") (roundrect_rratio 0.217391)
+    (pad "2" smd roundrect (at 1.475 0 90) (size 1.15 1.8) (layers "B.Cu" "B.Paste" "B.Mask") (roundrect_rratio 0.2173913043)
       (net 2 "GND") (pintype "passive"))
     (model "${KICAD6_3DMODEL_DIR}/Capacitor_SMD.3dshapes/C_1206_3216Metric.wrl"
@@
     (fp_line (start 1.6 0.8) (end 1.6 -0.8)
       (stroke (width 0.1) (type solid)) (layer "B.Fab"))
-    (pad "1" smd roundrect (at -1.4625 0 270) (size 1.125 1.75) (layers "B.Cu" "B.Paste" "B.Mask") (roundrect_rratio 0.222222)
+    (pad "1" smd roundrect (at -1.4625 0 270) (size 1.125 1.75) (layers "B.Cu" "B.Paste" "B.Mask") (roundrect_rratio 0.2222222222)
       (net 1 "Net-(C1-Pad1)") (pintype "passive"))
-    (pad "2" smd roundrect (at 1.4625 0 270) (size 1.125 1.75) (layers "B.Cu" "B.Paste" "B.Mask") (roundrect_rratio 0.222222)
+    (pad "2" smd roundrect (at 1.4625 0 270) (size 1.125 1.75) (layers "B.Cu" "B.Paste" "B.Mask") (roundrect_rratio 0.2222222222)
       (net 3 "Net-(R11-Pad2)") (pintype "passive"))
     (model "${KICAD6_3DMODEL_DIR}/Resistor_SMD.3dshapes/R_1206_3216Metric.wrl"
@@
   (gr_line (start 170.522266 141.365008) (end 170.62361 141.066725)
     (stroke (width 0.264583) (type solid)) (layer "Edge.Cuts"))
-  (gr_text "v1.0.0" (at 125.75 132.4 110) (layer "B.Cu")
+  (gr_text "v1.1.0" (at 126 131.85 108) (layer "B.Cu")
     (effects (font (size 0.8 0.8) (thickness 0.15)) (justify mirror))
   )
-  (gr_text "AVANT" (at 124.05 125.05 97) (layer "B.Cu")
+  (gr_text "BAER" (at 124.35 124.2 95) (layer "B.Cu")
     (effects (font (size 0.8 0.8) (thickness 0.15)) (justify mirror))
   )
-  (gr_text "2023" (at 124.65 128.75 103) (layer "B.Cu")
+  (gr_text "2023" (at 124.9 127.9 101) (layer "B.Cu")
     (effects (font (size 0.8 0.8) (thickness 0.15)) (justify mirror))
   )
-  (gr_text "FOR" (at 123.75 121.7 92) (layer "B.Cu")
+  (gr_text "MOSER" (at 124.1 120.05 92) (layer "B.Cu")
     (effects (font (size 0.8 0.8) (thickness 0.15)) (justify mirror))
   )
@@
   (zone (net 2) (net_name "GND") (layers "F&B.Cu") (hatch edge 0.508)
     (connect_pads (clearance 0.3))
-    (min_thickness 0.3) (filled_areas_thickness no)
-    (fill yes (thermal_gap 0.3) (thermal_bridge_width 0.5))
+    (min_thickness 0.2) (filled_areas_thickness no)
+    (fill yes (thermal_gap 0.3) (thermal_bridge_width 0.2))
     (polygon
       (pts
